File: Eagle Files/antenna_tracker.sch (EAGLE design)
At the start: 90 parts, among them IC1 ATMEGA1280-16AU, IC2 L298, Q11 BSS138, Q12 BSS138, Q8 16MHz, U1 LSM303DLHC, U2 MIC5219-3.3V, U4 FT232RL-BASICSSOP, U5 LD1117, X2 KUSBVX-BS1N

Commit message: Switched to 9DOF IC and a new 7.2V Buck Convertor
Added LSM9DS0 and MC34063
Parts:
- removed C1: 10µF, microbuilder:CAP_CERAMIC_0805
- removed C2: 0.1uF, rcl:C-EUC0603K
- removed C4: 4.70µF, microbuilder:CAP_CERAMIC_0805
- removed C5: 0.22µF, microbuilder:CAP_CERAMIC_0805
- removed NR6028: 4.7uH, resistor:L-USWE-TPC
- removed R3: 50k, rcl:R-US_M0805
- removed R5: 6.34k, rcl:R-US_M0805
- removed RB056L: (no value), diode:DIODE-DO214AC
- removed U$18: DF13-5P-1.25DSA, pixhawk2:DF13-5P-1.25DSA
- removed U$3: AP3211, antenna_tracker:AP3211
- removed U1: LSM303DLHC, microbuilder:LSM303DLHC
- added C16: 270pF, resistor:C-EUC0603K
- added C20: 100uF, rcl:CPOL-USE2,5-6E
- added C21: 470uF, rcl:CPOL-USE3.5-8
- added C28: 10uF, SparkFun-Capacitors:10UF-16V-10%(TANT)
- added D10: 1N5819, diode:DIODE-SOD123
- added IC3: MC34063AD, mc34063:MC34063AD
- added J203: DF13C-6P-1.25V, con-hirose-df13:DF13-6P-1.25V
- added L2: 15uH, rcl:L-USWE-TPC
- added R6: 0.20R, rcl:R-US_R0603
- added R7: 820R, resistor:R-US_R0603
- added R8: 3.9K, rcl:R-US_R0603
- added U6: LSM9DS0, SparkFun-DigitalIC:LSM9DS0
- C10, C9: device SparkFun:CAP0402-CAP -> resistor:C-EUC0603K; PARTNO (none) -> GRM188R71E104KA01D
- C11: value 10uF -> 0.22uF; device rcl:C-EUC0805K -> SparkFun-Capacitors:0.22UF-25V-10%(0603); PARTNO (none) -> CL10B224KA8NNNC
- C12: value 10nF -> 4.7uF; device rcl:C-EUC0603K -> SparkFun-Capacitors:4.7UF-6.3V-10%(0603)0603; PARTNO (none) -> CL10B475KQ8NQNC
- C13, C15: PARTNO (none) -> CL21A106KAFN3NE
- C14: value 22uF -> 1.0uF; device rcl:C-EUC0603K -> SparkFun-Capacitors:1.0UF-16V-10%(0603); PARTNO (none) -> C0603C105K8PACTU
- C17, C18, C23, C24, C25, C26, C27, C3: PARTNO (none) -> GRM188R71E104KA01D
- C19, C22: PARTNO (none) -> C0805C220J5GACTU
- C6: PARTNO (none) -> C0603C105K8PACTU
- C7: PARTNO (none) -> GRM1555C1H471JA01D
- C8: PARTNO (none) -> EEE-1CA100SR
- CHRG/LBO5: PARTNO (none) -> APT2012SECK
- D1, D2, D3, D4, D5, D6, D7, D8: PARTNO (none) -> ES2B-LTP
- F2: PARTNO (none) -> RUEF700-2
- ICSP: PARTNO (none) -> PPTC032LFBN-RC
- J$1: PARTNO (none) -> 0732511150
- JP1, SV1, SV3: PARTNO (none) -> PREC040SFAN-RC
- L4, L5: PARTNO (none) -> BLM15HD102SN1D
- L6: PARTNO (none) -> BKP1005HS121-T
- LED1: device SparkFun:LED0603 -> led:LEDCHIP-LED0805; PARTNO (none) -> LG R971-KN-1
- LED2: device SparkFun:LED0603 -> led:LEDCHIP-LED0805; PARTNO (none) -> LH R974-LP-1
- LED3, LED4: value (none) -> Orange; PARTNO (none) -> APT2012SECK
- Q11, Q12: PARTNO (none) -> BSS138
- Q8: PARTNO (none) -> ATS16B
- R1, R2: PARTNO (none) -> MCR01MRTF3300
- R16, R23, R24, R31, R32: PARTNO (none) -> 1623097-1
- R33: PARTNO (none) -> RMCF0805JT1K00
- R4: value (none) -> 1k; device resistor:R-US_R0603 -> resistor:R-US_R0805; PARTNO (none) -> RMCF0805JT1K00
- S1: PARTNO (none) -> 1825261-2
- S2: PARTNO (none) -> 1825910-6
- U$10, U$11: PARTNO (none) -> RCJ-021
- U2: PARTNO (none) -> MIC5219-3.3YM5 TR
- U4: PARTNO (none) -> FT232RL-REEL
- U5: PARTNO (none) -> LD1117DT50CTR
- X1, X10, X3, X4, X6, X7, X8: PARTNO (none) -> OSTTC022162
- X2: PARTNO (none) -> 5787834-1
Connections:
- removed net DRDY: U1.DRDY
- removed net INT1: U1.INT1
- removed net INT2: U1.INT2
- removed net N$1: C5.P$2, U1.SETC
- removed net N$3: C4.P$2, U1.C1
- removed net N$4: C5.P$1, U1.SETP
- new net DEN_G: U6.DEN(G)
- new net DRDY_G: U6.DRDY(G)
- new net INT1_XM: U6.INT1(XM)
- new net INT2_XM: U6.INT2(XM)
- new net INT_G: U6.INT(G)
- new net N$19: C16.1, IC3.TC
- new net N$30: IC3.DC, IC3.IS, IC3.SWC, R6.1
- new net N$31: IC3.FB, R7.2, R8.2
- new net N$32: D10.C, IC3.SWE, L2.1
- net +12V: now also C20.+, IC3.VCC, R6.2; no longer C11.1, U$3.EN, U$3.IN
- net +3V3: now also C14.1, C28.+, U6.CS(G), U6.CS(XM), U6.SDO(G), U6.SDO(XM), U6.VDD, U6.VDD_IO; no longer C1.P$1, C2.1, U1.VDD, U1.VDDIO
- net +5V: now also J203.2; no longer U$18-1.S
- net +7V: now also C21.+, L2.2, R8.1; no longer C14.2, NR6028.2, R3.2
- net GND: now also C12.2, C14.2, C16.2, C20.-, C21.-, C28.-, D10.A, IC3.GND, J203.1, J203.5, R7.1, U6.GND; no longer C1.P$2, C11.2, C14.1, C2.2, C4.P$1, R5.1, RB056L.A, U$18-5.S, U$3.GND, U1.GND@1, U1.GND@2, U1.GND@3
- net N$28: now also C11.2, U6.SETC; no longer C12.2, NR6028.1, RB056L.C, U$3.SW
- net N$29: now also C12.1, U6.C1; no longer R3.1, R5.2, U$3.FB
- net N$7: now also C11.1, U6.SETP; no longer C12.1, U$3.BS
- net RX1: now also J203.4; no longer U$18-3.S
- net SCL: now also U6.SCL; no longer U1.SCL
- net SDA: now also U6.SDA; no longer U1.SDA
- net TX1: now also J203.3; no longer U$18-2.S
